Commit message: Feat: use openvino yolo

File: src/hunter_se_description/urdf/hunter_se_description.urdf (robot description, URDF)
Before this commit: robot hunter_se_description, 9 links, 8 joints
Links:
- added link base_footprint
Joints:
- added joint base_footprint_joint: type fixed, parent base_footprint, child base_link, origin xyz=0 0 0 rpy=0 0 0

File: src/hunter_se_description/urdf/hunter_se_description.xacro (robot description, xacro)
@@ -9,4 +9,10 @@
 <robot
   name="hunter_se_description_2">
+  <link name="base_footprint"/>
+  <joint name="base_footprint_joint" type="fixed">
+    <parent link="base_footprint"/>
+    <child link="base_link"/>
+    <origin xyz="0 0 0" rpy="0 0 0"/>
+  </joint>
   <link
     name="base_link">
